File: eagle/NoiseGen_1.sch (EAGLE design)
At the start: 35 parts, among them Q1 BC337, Q2 BC327, U1 NE5532, U2 NE5532

Commit message: updating schematic
Parts:
- removed U$9: 4k7, RZEDKA_2017:TRIMMER1
- added R13: 4k7, rcl:R-EU_R0805
Connections:
- net N$12: now also R13.2; no longer U$9.A
- net OUT: now also R13.1; no longer U$9.E, U$9.S
Other:
- note added: "15.4 kHz"
Changed lines of the file:
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@@
 <part name="GND1" library="supply1" library_urn="urn:adsk.eagle:library:371" deviceset="GND" device=""/>
 <part name="GND2" library="supply1" library_urn="urn:adsk.eagle:library:371" deviceset="GND" device=""/>
-<part name="U$9" library="RZEDKA_2017" deviceset="TRIMMER1" device="" value="4k7"/>
 <part name="Q1" library="transistor" library_urn="urn:adsk.eagle:library:402" deviceset="BC337" device="" package3d_urn="urn:adsk.eagle:package:28523/2"/>
 <part name="Q2" library="transistor-pnp" library_urn="urn:adsk.eagle:library:399" deviceset="BC327" device="" package3d_urn="urn:adsk.eagle:package:29211/2"/>
@@
 <part name="GND5" library="supply1" library_urn="urn:adsk.eagle:library:371" deviceset="GND" device=""/>
 <part name="GND6" library="supply1" library_urn="urn:adsk.eagle:library:371" deviceset="GND" device=""/>
+<part name="R13" library="rcl" library_urn="urn:adsk.eagle:library:334" deviceset="R-EU_" device="R0805" package3d_urn="urn:adsk.eagle:package:23553/2" value="4k7"/>
 </parts>
 <sheets>
@@
 <text x="251.46" y="93.98" size="1.778" layer="91">0 - 4 Vpp</text>
 <text x="251.46" y="88.9" size="1.778" layer="91">0 - 666 mVrms</text>
+<text x="231.14" y="76.2" size="1.778" layer="91">15.4 kHz</text>
 </plain>
 <instances>
@@
 <attribute name="VALUE" x="35.56" y="-10.16" size="1.778" layer="96"/>
 </instance>
-<instance part="U$9" gate="G$1" x="228.6" y="83.82" smashed="yes" rot="R270">
-<attribute name="NAME" x="229.87" y="86.995" size="1.778" layer="95"/>
-<attribute name="VALUE" x="230.886" y="81.026" size="1.778" layer="96"/>
-</instance>
 <instance part="Q1" gate="G$1" x="-33.02" y="53.34" smashed="yes">
 <attribute name="NAME" x="-35.56" y="58.42" size="1.778" layer="95"/>
@@
 <instance part="GND6" gate="1" x="-55.88" y="-7.62" smashed="yes">
 <attribute name="VALUE" x="-58.42" y="-10.16" size="1.778" layer="96"/>
+</instance>
+<instance part="R13" gate="G$1" x="228.6" y="83.82" smashed="yes" rot="R180">
+<attribute name="NAME" x="232.41" y="82.3214" size="1.778" layer="95" rot="R180"/>
+<attribute name="VALUE" x="232.41" y="87.122" size="1.778" layer="96" rot="R180"/>
 </instance>
 </instances>
@@
 <wire x1="215.9" y1="73.66" x2="210.82" y2="73.66" width="0.1524" layer="91"/>
 <junction x="210.82" y="73.66"/>
-<pinref part="U$9" gate="G$1" pin="A"/>
+<pinref part="R13" gate="G$1" pin="2"/>
 <wire x1="223.52" y1="83.82" x2="210.82" y2="83.82" width="0.1524" layer="91"/>
 <junction x="210.82" y="83.82"/>
@@
 <wire x1="243.84" y1="83.82" x2="243.84" y2="91.44" width="0.1524" layer="91"/>
 <wire x1="231.14" y1="91.44" x2="243.84" y2="91.44" width="0.1524" layer="91"/>
-<pinref part="U$9" gate="G$1" pin="E"/>
-<wire x1="233.68" y1="83.82" x2="236.22" y2="83.82" width="0.1524" layer="91"/>
 <junction x="243.84" y="83.82"/>
-<pinref part="U$9" gate="G$1" pin="S"/>
-<wire x1="236.22" y1="83.82" x2="243.84" y2="83.82" width="0.1524" layer="91"/>
-<wire x1="228.6" y1="78.74" x2="236.22" y2="78.74" width="0.1524" layer="91"/>
-<wire x1="236.22" y1="78.74" x2="236.22" y2="83.82" width="0.1524" layer="91"/>
-<junction x="236.22" y="83.82"/>
+<wire x1="233.68" y1="83.82" x2="243.84" y2="83.82" width="0.1524" layer="91"/>
 <pinref part="V4" gate="G$1" pin="TP"/>
 <wire x1="248.92" y1="83.82" x2="243.84" y2="83.82" width="0.1524" layer="91"/>
@@
 <junction x="243.84" y="68.58"/>
 <label x="258.318" y="69.85" size="1.778" layer="95"/>
-</segment>
-</net>
+<pinref part="R13" gate="G$1" pin="1"/>
+</segment>
+</net>
